File: pcb/motorboard.kicad_pcb (KiCad board)
At the start: 4 copper layers, 72 x 74.3 mm, 75 parts, among them J1 RJ45, J2 RJ45, J3 Conn_01x02_Pin, J4 BATT+, J6 THROTTLE, J7 BATT-, U1 XIAO-RP2350-SMD, U11 TLV76701DRVR, U2 TCAN1042HGVDQ1, U3 ISO7041FQDBQRQ1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

Commit message: basic firmware, CAN consumption -> DAC only, no frame format
Connections:
- C14 pad 2: Net-(D2-A) -> Net-(U5-FB)
- R10 pad 1: Net-(D2-A) -> Net-(U5-FB)
- R11 pad 2: Net-(D2-A) -> Net-(U5-FB)
- U5 pad 5: Net-(D2-A) -> Net-(U5-FB)
- U5 pad EPAD: GND2 -> (no net)
Routing:
- net Net-(U5-FB): track 0.00 -> 7.51 mm
- net Net-(D2-A): track 16.8 -> 9.30 mm
Changed lines of the file:
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@@
 	(net 48 "/SCK")
 	(net 49 "Net-(U4-VFB)")
+	(net 50 "Net-(U5-FB)")
 	(footprint "Resistor_SMD:R_0603_1608Metric"
 		(layer "F.Cu")
@@
 			(layers "F.Cu" "F.Paste" "F.Mask")
 			(roundrect_rratio 0.25)
-			(net 16 "Net-(D2-A)")
+			(net 50 "Net-(U5-FB)")
 			(pintype "passive")
 		)
@@
 			(layers "F.Cu" "F.Paste" "F.Mask")
 			(roundrect_rratio 0.25)
-			(net 16 "Net-(D2-A)")
+			(net 50 "Net-(U5-FB)")
 			(pintype "passive")
 		)
@@
 			(size 1.4605 0.5588)
 			(layers "F.Cu" "F.Paste" "F.Mask")
-			(net 16 "Net-(D2-A)")
+			(net 50 "Net-(U5-FB)")
 			(pinfunction "FB")
 			(pintype "input")
@@
 			(size 2.3876 3.0988)
 			(layers "F.Cu" "F.Mask")
-			(net 10 "GND2")
 		)
 	)
@@
 			(layers "F.Cu" "F.Paste" "F.Mask")
 			(roundrect_rratio 0.25)
-			(net 16 "Net-(D2-A)")
+			(net 50 "Net-(U5-FB)")
 			(pintype "passive")
 		)
@@
 	)
 	(segment
-		(start 153.523 64.597)
-		(end 151.426 64.597)
-		(width 0.508)
-		(layer "F.Cu")
-		(net 16)
-	)
-	(segment
-		(start 151.426 64.597)
-		(end 151.426 66.729)
-		(width 0.508)
-		(layer "F.Cu")
-		(net 16)
-	)
-	(segment
 		(start 157.551 72.712)
 		(end 157.551 73.6795)
@@
 		(net 16)
 	)
-	(segment
-		(start 151.426 63.681)
-		(end 151.426 64.597)
-		(width 0.381)
-		(layer "F.Cu")
-		(net 16)
-	)
-	(segment
-		(start 151.426 66.729)
-		(end 151.453 66.756)
-		(width 0.508)
-		(layer "F.Cu")
-		(net 16)
-	)
-	(segment
-		(start 151.453 66.756)
-		(end 153.78285 66.756)
-		(width 0.508)
-		(layer "F.Cu")
-		(net 16)
-	)
 	(via
 		(at 157.551 72.712)
@@
 		(net 49)
 	)
+	(segment
+		(start 153.523 64.597)
+		(end 151.426 64.597)
+		(width 0.508)
+		(layer "F.Cu")
+		(net 50)
+	)
+	(segment
+		(start 151.426 64.597)
+		(end 151.426 66.729)
+		(width 0.508)
+		(layer "F.Cu")
+		(net 50)
+	)
+	(segment
+		(start 151.426 63.681)
+		(end 151.426 64.597)
+		(width 0.381)
+		(layer "F.Cu")
+		(net 50)
+	)
+	(segment
+		(start 151.426 66.729)
+		(end 151.453 66.756)
+		(width 0.508)
+		(layer "F.Cu")
+		(net 50)
+	)
+	(segment
+		(start 151.453 66.756)
+		(end 153.78285 66.756)
+		(width 0.508)
+		(layer "F.Cu")
+		(net 50)
+	)
 	(zone
