File: pcb/motorboard.kicad_sch (KiCad schematic)
At the start: 25 parts, among them J6 THROTTLE, U1 XIAO-RP2350-SMD, U3 ISO7041FQDBQRQ1, U4 DAC6551AQDGKRQ1, U6 TLV9361QDBVRQ1, U7 TLV76701DRVR, U8 TLV76701DRVR

Commit message: basic firmware, CAN consumption -> DAC only, no frame format
Other:
- note added: "Vout = 1.515 (3.3) = 5 V"
- note added: "Vout = Vin (1 + Rf/R2) = Vin (1+0.515) = 1.515*Vin"
- note removed: "Vout = 3.06 (3.3) = 10.01 V"
- note removed: "Vout = Vin (1 + Rf/R2) = Vin (1+2.06) = 3.06 Vin"
Changed lines of the file:
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@@
 		)
 	)
-	(text "Vout = 3.06 (3.3) = 10.01 V\n"
+	(text "Vout = 1.515 (3.3) = 5 V\n"
 		(exclude_from_sim no)
 		(at 171.196 137.922 0)
@@
 		)
 	)
-	(text "Vout = Vin (1 + Rf/R2) = Vin (1+2.06) = 3.06 Vin"
+	(text "Vout = Vin (1 + Rf/R2) = Vin (1+0.515) = 1.515*Vin\n"
 		(exclude_from_sim no)
 		(at 182.372 134.366 0)
